File: doc/Boards/ConnectBoard/elec/ConnectBoard/ConnectBoard.sch (KiCad schematic (older format))
At the start: 4 parts, among them J1 Sonar0, J2 PowerSelect0, J3 PropEdgeConnect-Conn1

Commit message: WIP
Parts:
- added PropEdgeConnect-Conn2: PropEdgeConnect-Conn2, Connector_PinSocket_2.54mm:PinSocket_2x06_P2.54mm_Vertical, symbol Connector_Generic:Conn_02x06_Top_Bottom
- added PropEdgeConnect-Conn3: PropEdgeConnect-Conn3, Connector_PinSocket_2.54mm:PinSocket_2x06_P2.54mm_Vertical, symbol Connector_Generic:Conn_02x06_Top_Bottom
- added R2, R3, R4: 4.7k, Resistor_THT:R_Axial_DIN0207_L6.3mm_D2.5mm_P7.62mm_Horizontal, symbol Device:R
- added S1, S2, S3: S0, Connector_PinHeader_2.54mm:PinHeader_1x03_P2.54mm_Vertical, symbol Connector:Conn_01x03_Male
- S0: renamed from J1; value Sonar0 -> S0
- renumbered J2 to PowerSelect0, J3 to PropEdgeConnect-Conn1
Connections:
- net GND: now also S1.3 (Pin_3), S2.3 (Pin_3), S3.3 (Pin_3)
- net at PowerSelect0.2 (Pin_2), S0.2 (Pin_2): now also S1.2 (Pin_2), S2.2 (Pin_2), S3.2 (Pin_2)
- net P2: now reaches PropEdgeConnect-Conn1.3 (Pin_3)
- net P2: now also R2.1
- net P4: now reaches PropEdgeConnect-Conn1.4 (Pin_4)
- net P4: now also R3.1
- net P6: now reaches PropEdgeConnect-Conn1.5 (Pin_5)
- net P6: now also R4.1
- new net: R2.2, S1.1 (Pin_1)
- new net: R3.2, S2.1 (Pin_1)
- new net: R4.2, S3.1 (Pin_1)
- no-connect marks 7 -> 28

Commit message: WIP
Parts:
- added R5, R6, R7, R8: 4.7k, Resistor_THT:R_Axial_DIN0207_L6.3mm_D2.5mm_P7.62mm_Horizontal, symbol Device:R
- added S1, S3, S5, S7: SonarConnect, Connector_PinHeader_2.54mm:PinHeader_1x03_P2.54mm_Vertical, symbol Connector:Conn_01x03_Male
- PS0: renamed from PowerSelect0; value PowerSelect0 -> PowerSelect
- S0: value S0 -> SonarConnect
- S2: renamed from S1; value S0 -> SonarConnect
- S4: renamed from S2; value S0 -> SonarConnect
- S6: renamed from S3; value S0 -> SonarConnect
Connections:
- net GND: now also S1.3 (Pin_3), S3.3 (Pin_3), S5.3 (Pin_3), S7.3 (Pin_3)
- net at PS0.2 (Pin_2), S0.2 (Pin_2), S2.2 (Pin_2)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: now also S1.2 (Pin_2), S3.2 (Pin_2), S5.2 (Pin_2), S7.2 (Pin_2)
- net P5: now reaches PropEdgeConnect-Conn1.10 (Pin_10)
- net P5: now also R7.2
- net P7: now reaches PropEdgeConnect-Conn1.11 (Pin_11)
- net P7: now also R8.2
- net P1: now reaches PropEdgeConnect-Conn1.8 (Pin_8)
- net P1: now also R5.2
- net P3: now reaches PropEdgeConnect-Conn1.9 (Pin_9)
- net P3: now also R6.2
- new net: R5.1, S1.1 (Pin_1)
- new net: R6.1, S3.1 (Pin_1)
- new net: R7.1, S5.1 (Pin_1)
- new net: R8.1, S7.1 (Pin_1)
- no-connect marks 28 -> 24
Other:
- moved on the sheet: PS0, R1, R2, R3, R4, S0, S2, S4, S6
