File: doc/Boards/ConnectBoard/elec/ConnectBoard/ConnectBoard.sch (KiCad schematic (older format))
At the start: 20 parts

Commit message: Updates
Parts:
- removed PropEdgeConnect-Conn1: PropEdgeConnect-Conn1, Connector_PinSocket_2.54mm:PinSocket_2x06_P2.54mm_Vertical, symbol Connector_Generic:Conn_02x06_Top_Bottom
- removed PropEdgeConnect-Conn2: PropEdgeConnect-Conn2, Connector_PinSocket_2.54mm:PinSocket_2x06_P2.54mm_Vertical, symbol Connector_Generic:Conn_02x06_Top_Bottom
- removed PropEdgeConnect-Conn3: PropEdgeConnect-Conn3, Connector_PinSocket_2.54mm:PinSocket_2x06_P2.54mm_Vertical, symbol Connector_Generic:Conn_02x06_Top_Bottom
- added Conn1, Conn2, Conn3, Conn4: PropEdgeConnect, Connector_PinSocket_2.54mm:PinSocket_2x06_P2.54mm_Vertical, symbol Connector_Generic:Conn_02x06_Odd_Even
- added J1: Prop_CommPort, Connector_PinSocket_2.54mm:PinSocket_1x04_P2.54mm_Vertical, symbol Connector:Conn_01x04_Male
- added PS2, PS3: PowerSelect, Connector_PinHeader_2.54mm:PinHeader_1x03_P2.54mm_Vertical, symbol Connector:Conn_01x03_Male
- added R1, R10, R11, R12, R17, R18, R19, R2, R20, R3, R4, R5, R6, R7, R8, R9: 4.7k, Resistor_THT:R_Axial_DIN0207_L6.3mm_D2.5mm_P7.62mm_Horizontal, symbol Device:R
- added S1, S10, S11, S12, S17, S18, S19, S2, S20, S3, S4, S5, S6, S7, S8, S9: SonarConnect, Connector_PinHeader_2.54mm:PinHeader_1x03_P2.54mm_Vertical, symbol Connector:Conn_01x03_Male
- renumbered PS0 to PS1, R1 to R13, R2 to R14, R3 to R15, R4 to R16, R5 to R21, R6 to R22, R7 to R23, R8 to R24, S0 to S13, S2 to S14, S4 to S15, S6 to S16, S1 to S21, S3 to S22, S5 to S23, S7 to S24
Connections:
- net P1 is gone; now on an unnamed net: R21.2
- net P3 is gone; now on an unnamed net: R22.2
- net P5 is gone; now on an unnamed net: R23.2
- net P7 is gone; now on an unnamed net: R24.2
- net GND: now also Conn1.1 (Pin_1), Conn1.2 (Pin_2), Conn2.11 (Pin_11), Conn2.12 (Pin_12), Conn3.11 (Pin_11), Conn3.12 (Pin_12), Conn4.11 (Pin_11), Conn4.12 (Pin_12), J1.4 (Pin_4), S1.3 (Pin_3), S10.3 (Pin_3), S11.3 (Pin_3), S12.3 (Pin_3), S17.3 (Pin_3), S18.3 (Pin_3), S19.3 (Pin_3), S2.3 (Pin_3), S20.3 (Pin_3), S3.3 (Pin_3), S4.3 (Pin_3), S5.3 (Pin_3), S6.3 (Pin_3), S7.3 (Pin_3), S8.3 (Pin_3), S9.3 (Pin_3)
- net P0: now also Conn1.3 (Pin_3), J1.1 (Pin_1); no longer R13.1
- net P2: now also Conn1.5 (Pin_5), J1.2 (Pin_2); no longer R14.1
- net at S21.1 (Pin_1): no longer R21.1
- net at S22.1 (Pin_1): no longer R22.1
- net at S23.1 (Pin_1): no longer R23.1
- net at S24.1 (Pin_1): no longer R24.1
- net +3V3 renamed V56
- net V56: now also Conn2.1 (Pin_1)
- net +5V renamed +5V1
- net +5V1: now also Conn3.2 (Pin_2), PS2.3 (Pin_3)
- net P4 renamed P59
- net P59: now also Conn2.7 (Pin_7)
- net P6 renamed P57
- net P57: now also Conn2.9 (Pin_9)
- new net: R1.2, S1.1 (Pin_1)
- new net: PS2.2 (Pin_2), S1.2 (Pin_2), S2.2 (Pin_2), S3.2 (Pin_2), S4.2 (Pin_2), S5.2 (Pin_2), S6.2 (Pin_2), S7.2 (Pin_2), S8.2 (Pin_2)
- new net: R2.2, S2.1 (Pin_1)
- new net: R3.2, S3.1 (Pin_1)
- new net: R4.2, S4.1 (Pin_1)
- new net: R5.1, S5.1 (Pin_1)
- new net: R6.1, S6.1 (Pin_1)
- new net: R7.1, S7.1 (Pin_1)
- new net: R8.1, S8.1 (Pin_1)
- new net: R9.2, S9.1 (Pin_1)
- new net: PS3.2 (Pin_2), S10.2 (Pin_2), S11.2 (Pin_2), S12.2 (Pin_2), S17.2 (Pin_2), S18.2 (Pin_2), S19.2 (Pin_2), S20.2 (Pin_2), S9.2 (Pin_2)
- new net: R10.2, S10.1 (Pin_1)
- new net: R11.2, S11.1 (Pin_1)
- new net: R12.2, S12.1 (Pin_1)
- new net: R17.1, S17.1 (Pin_1)
- new net: R18.1, S18.1 (Pin_1)
- new net: R19.1, S19.1 (Pin_1)
- new net: R20.1, S20.1 (Pin_1)
- new net +5V0: Conn1.11 (Pin_11)
- new net +5V3: Conn4.2 (Pin_2), PS3.3 (Pin_3)
- new net P40: Conn4.10 (Pin_10), R20.2
- new net P41: Conn4.9 (Pin_9), R12.1
- new net P42: Conn4.8 (Pin_8), R19.2
- new net P43: Conn4.7 (Pin_7), R11.1
- new net P44: Conn4.6 (Pin_6), R18.2
- new net P45: Conn4.5 (Pin_5), R10.1
- new net P46: Conn4.4 (Pin_4), R17.2
- new net P47: Conn4.3 (Pin_3), R9.1
- new net P48: Conn3.10 (Pin_10), R8.2
- new net P49: Conn3.9 (Pin_9), R4.1
- new net P50: Conn3.8 (Pin_8), R7.2
- new net P51: Conn3.7 (Pin_7), R3.1
- new net P52: Conn3.6 (Pin_6), R6.2
- new net P53: Conn3.5 (Pin_5), R2.1
- new net P54: Conn3.4 (Pin_4), R5.2
- new net P55: Conn3.3 (Pin_3), R1.1
- new net P56: Conn2.10 (Pin_10), R24.1
- new net P58: Conn2.8 (Pin_8), R23.1
- new net P60: Conn2.6 (Pin_6), R22.1
- new net P61: Conn2.5 (Pin_5), R14.1
- new net P62: Conn2.4 (Pin_4), R21.1
- new net P63: Conn2.3 (Pin_3), R13.1
- new net V00: Conn1.12 (Pin_12)
- new net V40: Conn4.1 (Pin_1), PS3.1 (Pin_1)
- new net V48: Conn3.1 (Pin_1), PS2.1 (Pin_1)
- no-connect marks 24 -> 8
Other:
- moved on the sheet: PS1, R13, R14, R15, R16, R21, R22, R23, R24, S13, S14, S15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

Commit message: More work on this.
Parts:
- removed R1, R10, R11, R12, R13, R14, R15, R16, R17, R18, R19, R2, R20, R21, R22, R23, R24, R3, R4, R5, R6, R7, R8, R9: 4.7k, Resistor_THT:R_Axial_DIN0207_L6.3mm_D2.5mm_P7.62mm_Horizontal, symbol Device:R
- added R1, R2: 4.7k, Package_DIP:DIP-8_W7.62mm, symbol Device:R_Pack04_Split
- added R3, R4, R5, R6: R_Pack04_Split, Package_DIP:DIP-8_W7.62mm, symbol Device:R_Pack04_Split
- J0: renamed from J1; footprint Connector_PinSocket_2.54mm:PinSocket_1x04_P2.54mm_Vertical -> Connector_PinHeader_2.54mm:PinHeader_1x04_P2.54mm_Vertical
- renumbered S24 to S1, S4 to S10, S7 to S11, S3 to S12, S6 to S13, S2 to S14, S5 to S15, S1 to S16, S20 to S17, S12 to S18, S16 to S2, S11 to S20, S18 to S21, S10 to S22, S17 to S23, S9 to S24, S23 to S3, S15 to S4, S22 to S5, S14 to S6, S21 to S7, S13 to S8, S8 to S9
Connections:
- net P40: now also R6.4
- net P41: now also R5.5
- net P42: now also R6.3
- net P43: now also R5.6
- net P44: now also R6.2
- net P45: now also R5.7
- net P46: now also R6.1
- net P47: now also R5.8
- net P48: now also R4.4
- net P49: now also R3.5
- net P50: now also R4.3
- net P51: now also R3.6
- net P52: now also R4.2
- net P53: now also R3.7
- net P54: now also R4.1
- net P55: now also R3.8
- net P56: now also R2.4
- net P57: now also R2.3
- net P58: now also R2.2
- net P59: now also R2.1
- net P60: now also R1.4
- net P61: now also R1.3
- net P62: now also R1.2
- net P63: now also R1.1
- net at S8.1 (Pin_1): now also R1.8
- net at S6.1 (Pin_1): now also R1.6
- net at S4.1 (Pin_1): now also R2.8
- net at S2.1 (Pin_1): now also R2.6
- net at S7.1 (Pin_1): now also R1.7
- net at S5.1 (Pin_1): now also R1.5
- net at S3.1 (Pin_1): now also R2.7
- net at S1.1 (Pin_1): now also R2.5
- net at S16.1 (Pin_1): now also R3.1
- net at S14.1 (Pin_1): now also R3.2
- net at S12.1 (Pin_1): now also R3.3
- net at S10.1 (Pin_1): now also R3.4
- net at S15.1 (Pin_1): now also R4.8
- net at S13.1 (Pin_1): now also R4.7
- net at S11.1 (Pin_1): now also R4.6
- net at S9.1 (Pin_1): now also R4.5
- net at S24.1 (Pin_1): now also R5.1
- net at S22.1 (Pin_1): now also R5.2
- net at S20.1 (Pin_1): now also R5.3
- net at S18.1 (Pin_1): now also R5.4
- net at S23.1 (Pin_1): now also R6.8
- net at S21.1 (Pin_1): now also R6.7
- net at S19.1 (Pin_1): now also R6.6
- net at S17.1 (Pin_1): now also R6.5

Commit message: Updates
Connections:
- net P40: now also R5.4; no longer R6.4
- net P41: now also R5.3; no longer R5.5
- net P42: now also R5.2; no longer R6.3
- net P43: now also R5.1; no longer R5.6
- net P44: now also R6.4; no longer R6.2
- net P45: now also R6.3; no longer R5.7
- net P46: now also R6.2; no longer R6.1
- net P47: now also R6.1; no longer R5.8
- net P48: now also R3.4; no longer R4.4
- net P49: now also R3.3; no longer R3.5
- net P50: now also R3.2; no longer R4.3
- net P51: now also R3.1; no longer R3.6
- net P52: now also R4.4; no longer R4.2
- net P53: now also R4.3; no longer R3.7
- net P54: now also R4.2; no longer R4.1
- net P55: now also R4.1; no longer R3.8
- net at S16.1 (Pin_1): now also R4.8; no longer R3.1
- net at S14.1 (Pin_1): now also R4.6; no longer R3.2
- net at S12.1 (Pin_1): now also R3.8; no longer R3.3
- net at S10.1 (Pin_1): now also R3.6; no longer R3.4
- net at S15.1 (Pin_1): now also R4.7; no longer R4.8
- net at S13.1 (Pin_1): now also R4.5; no longer R4.7
- net at S11.1 (Pin_1): now also R3.7; no longer R4.6
- net at S9.1 (Pin_1): now also R3.5; no longer R4.5
- net at S24.1 (Pin_1): now also R6.8; no longer R5.1
- net at S23.1 (Pin_1): now also R6.7; no longer R6.8
- net at S22.1 (Pin_1): now also R6.6; no longer R5.2
- net at S21.1 (Pin_1): now also R6.5; no longer R6.7
- net at S20.1 (Pin_1): now also R5.8; no longer R5.3
- net at S19.1 (Pin_1): now also R5.7; no longer R6.6
- net at S18.1 (Pin_1): now also R5.6; no longer R5.4
- net at S17.1 (Pin_1): now also R5.5; no longer R6.5
Other:
- moved on the sheet: R3A, R3B, R3C, R3D, R4A, R4B, R4C, R4D, R5A, R5B, R5C, R5D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
Changed lines of the file:
@@
 L Device:R_Pack04_Split R3
 U 1 1 67EC40B0
-P 1900 4550
-F 0 "R3" V 1693 4550 50  0000 C CNN
-F 1 "R_Pack04_Split" V 1784 4550 50  0000 C CNN
-F 2 "Package_DIP:DIP-8_W7.62mm" V 1830 4550 50  0001 C CNN
-F 3 "~" H 1900 4550 50  0001 C CNN
-	1    1900 4550
-	0    1    1    0
+P 1900 5800
+F 0 "R3" V 1693 5800 50  0000 C CNN
+F 1 "R_Pack04_Split" V 1784 5800 50  0000 C CNN
+F 2 "Package_DIP:DIP-8_W7.62mm" V 1830 5800 50  0001 C CNN
+F 3 "~" H 1900 5800 50  0001 C CNN
+	1    1900 5800
+	0    -1   -1   0
 $EndComp
 $Comp
 L Device:R_Pack04_Split R3
 U 2 1 67EC5970
-P 1900 5100
-F 0 "R3" V 1693 5100 50  0000 C CNN
-F 1 "R_Pack04_Split" V 1784 5100 50  0000 C CNN
-F 2 "Package_DIP:DIP-8_W7.62mm" V 1830 5100 50  0001 C CNN
-F 3 "~" H 1900 5100 50  0001 C CNN
-	2    1900 5100
+P 4350 5800
+F 0 "R3" V 4143 5800 50  0000 C CNN
+F 1 "R_Pack04_Split" V 4234 5800 50  0000 C CNN
+F 2 "Package_DIP:DIP-8_W7.62mm" V 4280 5800 50  0001 C CNN
+F 3 "~" H 4350 5800 50  0001 C CNN
+	2    4350 5800
 	0    1    1    0
 $EndComp
@@
 L Device:R_Pack04_Split R3
 U 3 1 67EC6315
-P 1900 5800
-F 0 "R3" V 1693 5800 50  0000 C CNN
-F 1 "R_Pack04_Split" V 1784 5800 50  0000 C CNN
-F 2 "Package_DIP:DIP-8_W7.62mm" V 1830 5800 50  0001 C CNN
-F 3 "~" H 1900 5800 50  0001 C CNN
-	3    1900 5800
-	0    1    1    0
-$EndComp
-$Comp
-L Device:R_Pack04_Split R3
-U 4 1 67EC6C90
 P 1900 6350
 F 0 "R3" V 1693 6350 50  0000 C CNN
@@
 F 2 "Package_DIP:DIP-8_W7.62mm" V 1830 6350 50  0001 C CNN
 F 3 "~" H 1900 6350 50  0001 C CNN
-	4    1900 6350
-	0    1    1    0
+	3    1900 6350
+	0    -1   -1   0
 $EndComp
 $Comp
-L Device:R_Pack04_Split R4
-U 1 1 67ECBCAE
-P 4350 4550
-F 0 "R4" V 4143 4550 50  0000 C CNN
-F 1 "R_Pack04_Split" V 4234 4550 50  0000 C CNN
-F 2 "Package_DIP:DIP-8_W7.62mm" V 4280 4550 50  0001 C CNN
-F 3 "~" H 4350 4550 50  0001 C CNN
-	1    4350 4550
-	0    1    1    0
-$EndComp
-$Comp
-L Device:R_Pack04_Split R4
-U 2 1 67ECD7B7
-P 4350 5100
-F 0 "R4" V 4143 5100 50  0000 C CNN
-F 1 "R_Pack04_Split" V 4234 5100 50  0000 C CNN
-F 2 "Package_DIP:DIP-8_W7.62mm" V 4280 5100 50  0001 C CNN
-F 3 "~" H 4350 5100 50  0001 C CNN
-	2    4350 5100
-	0    1    1    0
-$EndComp
-$Comp
-L Device:R_Pack04_Split R4
-U 3 1 67ECE332
-P 4350 5800
-F 0 "R4" V 4143 5800 50  0000 C CNN
-F 1 "R_Pack04_Split" V 4234 5800 50  0000 C CNN
-F 2 "Package_DIP:DIP-8_W7.62mm" V 4280 5800 50  0001 C CNN
-F 3 "~" H 4350 5800 50  0001 C CNN
-	3    4350 5800
-	0    1    1    0
-$EndComp
-$Comp
-L Device:R_Pack04_Split R4
-U 4 1 67ED0766
+L Device:R_Pack04_Split R3
+U 4 1 67EC6C90
 P 4350 6350
-F 0 "R4" V 4143 6350 50  0000 C CNN
+F 0 "R3" V 4143 6350 50  0000 C CNN
 F 1 "R_Pack04_Split" V 4234 6350 50  0000 C CNN
 F 2 "Package_DIP:DIP-8_W7.62mm" V 4280 6350 50  0001 C CNN
@@
 $EndComp
 $Comp
+L Device:R_Pack04_Split R4
+U 1 1 67ECBCAE
+P 1900 4550
+F 0 "R4" V 1693 4550 50  0000 C CNN
+F 1 "R_Pack04_Split" V 1784 4550 50  0000 C CNN
+F 2 "Package_DIP:DIP-8_W7.62mm" V 1830 4550 50  0001 C CNN
+F 3 "~" H 1900 4550 50  0001 C CNN
+	1    1900 4550
+	0    -1   -1   0
+$EndComp
+$Comp
+L Device:R_Pack04_Split R4
+U 2 1 67ECD7B7
+P 4350 4550
+F 0 "R4" V 4143 4550 50  0000 C CNN
+F 1 "R_Pack04_Split" V 4234 4550 50  0000 C CNN
+F 2 "Package_DIP:DIP-8_W7.62mm" V 4280 4550 50  0001 C CNN
+F 3 "~" H 4350 4550 50  0001 C CNN
+	2    4350 4550
+	0    1    1    0
+$EndComp
+$Comp
+L Device:R_Pack04_Split R4
+U 3 1 67ECE332
+P 1900 5100
+F 0 "R4" V 1693 5100 50  0000 C CNN
+F 1 "R_Pack04_Split" V 1784 5100 50  0000 C CNN
+F 2 "Package_DIP:DIP-8_W7.62mm" V 1830 5100 50  0001 C CNN
+F 3 "~" H 1900 5100 50  0001 C CNN
+	3    1900 5100
+	0    -1   -1   0
+$EndComp
+$Comp
+L Device:R_Pack04_Split R4
+U 4 1 67ED0766
+P 4350 5100
+F 0 "R4" V 4143 5100 50  0000 C CNN
+F 1 "R_Pack04_Split" V 4234 5100 50  0000 C CNN
+F 2 "Package_DIP:DIP-8_W7.62mm" V 4280 5100 50  0001 C CNN
+F 3 "~" H 4350 5100 50  0001 C CNN
+	4    4350 5100
+	0    1    1    0
+$EndComp
+$Comp
 L Device:R_Pack04_Split R5
 U 1 1 67EDF60B
+P 6950 5550
+F 0 "R5" V 6743 5550 50  0000 C CNN
+F 1 "R_Pack04_Split" V 6834 5550 50  0000 C CNN
+F 2 "Package_DIP:DIP-8_W7.62mm" V 6880 5550 50  0001 C CNN
+F 3 "~" H 6950 5550 50  0001 C CNN
+	1    6950 5550
+	0    -1   -1   0
+$EndComp
+$Comp
+L Device:R_Pack04_Split R6
+U 1 1 67EDFF2D
 P 6950 4300
-F 0 "R5" V 6743 4300 50  0000 C CNN
+F 0 "R6" V 6743 4300 50  0000 C CNN
 F 1 "R_Pack04_Split" V 6834 4300 50  0000 C CNN
 F 2 "Package_DIP:DIP-8_W7.62mm" V 6880 4300 50  0001 C CNN
 F 3 "~" H 6950 4300 50  0001 C CNN
 	1    6950 4300
+	0    -1   -1   0
+$EndComp
+$Comp
+L Device:R_Pack04_Split R5
+U 2 1 67EE0C8C
+P 9400 5550
+F 0 "R5" V 9193 5550 50  0000 C CNN
+F 1 "R_Pack04_Split" V 9284 5550 50  0000 C CNN
+F 2 "Package_DIP:DIP-8_W7.62mm" V 9330 5550 50  0001 C CNN
+F 3 "~" H 9400 5550 50  0001 C CNN
+	2    9400 5550
 	0    1    1    0
 $EndComp
 $Comp
 L Device:R_Pack04_Split R6
-U 1 1 67EDFF2D
+U 2 1 67EE135C
 P 9400 4300
 F 0 "R6" V 9193 4300 50  0000 C CNN
@@
 F 2 "Package_DIP:DIP-8_W7.62mm" V 9330 4300 50  0001 C CNN
 F 3 "~" H 9400 4300 50  0001 C CNN
-	1    9400 4300
-	0    1    1    0
-$EndComp
-$Comp
-L Device:R_Pack04_Split R5
-U 2 1 67EE0C8C
-P 6950 4850
-F 0 "R5" V 6743 4850 50  0000 C CNN
-F 1 "R_Pack04_Split" V 6834 4850 50  0000 C CNN
-F 2 "Package_DIP:DIP-8_W7.62mm" V 6880 4850 50  0001 C CNN
-F 3 "~" H 6950 4850 50  0001 C CNN
-	2    6950 4850
-	0    1    1    0
-$EndComp
-$Comp
-L Device:R_Pack04_Split R6
-U 2 1 67EE135C
-P 9400 4850
-F 0 "R6" V 9193 4850 50  0000 C CNN
-F 1 "R_Pack04_Split" V 9284 4850 50  0000 C CNN
-F 2 "Package_DIP:DIP-8_W7.62mm" V 9330 4850 50  0001 C CNN
-F 3 "~" H 9400 4850 50  0001 C CNN
-	2    9400 4850
+	2    9400 4300
 	0    1    1    0
 $EndComp
@@
 L Device:R_Pack04_Split R5
 U 3 1 67EE1F05
-P 6950 5550
-F 0 "R5" V 6743 5550 50  0000 C CNN
-F 1 "R_Pack04_Split" V 6834 5550 50  0000 C CNN
-F 2 "Package_DIP:DIP-8_W7.62mm" V 6880 5550 50  0001 C CNN
-F 3 "~" H 6950 5550 50  0001 C CNN
-	3    6950 5550
-	0    1    1    0
-$EndComp
-$Comp
-L Device:R_Pack04_Split R6
-U 3 1 67EE27AF
-P 9400 5550
-F 0 "R6" V 9193 5550 50  0000 C CNN
-F 1 "R_Pack04_Split" V 9284 5550 50  0000 C CNN
-F 2 "Package_DIP:DIP-8_W7.62mm" V 9330 5550 50  0001 C CNN
-F 3 "~" H 9400 5550 50  0001 C CNN
-	3    9400 5550
-	0    1    1    0
-$EndComp
-$Comp
-L Device:R_Pack04_Split R5
-U 4 1 67EE34D7
 P 6950 6100
 F 0 "R5" V 6743 6100 50  0000 C CNN
@@
 F 2 "Package_DIP:DIP-8_W7.62mm" V 6880 6100 50  0001 C CNN
 F 3 "~" H 6950 6100 50  0001 C CNN
-	4    6950 6100
-	0    1    1    0
+	3    6950 6100
+	0    -1   -1   0
 $EndComp
 $Comp
 L Device:R_Pack04_Split R6
-U 4 1 67EE3CA6
+U 3 1 67EE27AF
+P 6950 4850
+F 0 "R6" V 6743 4850 50  0000 C CNN
+F 1 "R_Pack04_Split" V 6834 4850 50  0000 C CNN
+F 2 "Package_DIP:DIP-8_W7.62mm" V 6880 4850 50  0001 C CNN
+F 3 "~" H 6950 4850 50  0001 C CNN
+	3    6950 4850
+	0    -1   -1   0
+$EndComp
+$Comp
+L Device:R_Pack04_Split R5
+U 4 1 67EE34D7
 P 9400 6100
-F 0 "R6" V 9193 6100 50  0000 C CNN
+F 0 "R5" V 9193 6100 50  0000 C CNN
 F 1 "R_Pack04_Split" V 9284 6100 50  0000 C CNN
 F 2 "Package_DIP:DIP-8_W7.62mm" V 9330 6100 50  0001 C CNN
@@
 	0    1    1    0
 $EndComp
+$Comp
+L Device:R_Pack04_Split R6
+U 4 1 67EE3CA6
+P 9400 4850
+F 0 "R6" V 9193 4850 50  0000 C CNN
+F 1 "R_Pack04_Split" V 9284 4850 50  0000 C CNN
+F 2 "Package_DIP:DIP-8_W7.62mm" V 9330 4850 50  0001 C CNN
+F 3 "~" H 9400 4850 50  0001 C CNN
+	4    9400 4850
+	0    1    1    0
+$EndComp

Commit message: WIP
Connections:
- net GND: now also J0.1 (Pin_1); no longer J0.4 (Pin_4)
- net P0: now also J0.3 (Pin_3); no longer J0.1 (Pin_1)
- net P2: now also J0.4 (Pin_4); no longer J0.2 (Pin_2)
Other:
- moved on the sheet: J0
Changed lines of the file:
@@
 L Connector:Conn_01x04_Male J0
 U 1 1 67F6CA92
-P 1000 1250
-F 0 "J0" H 1108 1531 50  0000 C CNN
-F 1 "Prop_CommPort" H 1108 1440 50  0000 C CNN
-F 2 "Connector_PinHeader_2.54mm:PinHeader_1x04_P2.54mm_Vertical" H 1000 1250 50  0001 C CNN
-F 3 "~" H 1000 1250 50  0001 C CNN
-	1    1000 1250
+P 1000 1050
+F 0 "J0" H 1100 1300 50  0000 C CNN
+F 1 "Prop_CommPort" H 1150 750 50  0000 C CNN
+F 2 "Connector_PinHeader_2.54mm:PinHeader_1x04_P2.54mm_Vertical" H 1000 1050 50  0001 C CNN
+F 3 "~" H 1000 1050 50  0001 C CNN
+	1    1000 1050
 	1    0    0    -1
 $EndComp
@@
 Text Label 2600 1150 0    50   ~ 0
 P0
-NoConn ~ 1200 1350
+NoConn ~ 1200 1050
 $Comp
 L power:GND #PWR0112
 U 1 1 67F955D8
-P 1300 1550
-F 0 "#PWR0112" H 1300 1300 50  0001 C CNN
-F 1 "GND" V 1200 1550 50  0000 R CNN
-F 2 "" H 1300 1550 50  0001 C CNN
-F 3 "" H 1300 1550 50  0001 C CNN
-	1    1300 1550
-	1    0    0    -1
-$EndComp
-Wire Wire Line
-	1200 1450 1300 1450
-Wire Wire Line
-	1300 1450 1300 1550
+P 1300 950
+F 0 "#PWR0112" H 1300 700 50  0001 C CNN
+F 1 "GND" V 1200 950 50  0000 R CNN
+F 2 "" H 1300 950 50  0001 C CNN
+F 3 "" H 1300 950 50  0001 C CNN
+	1    1300 950
+	0    -1   -1   0
+$EndComp
 Text GLabel 8900 800  1    50   Input ~ 0
 V56
@@
 	0    1    1    0
 $EndComp
+Wire Wire Line
+	1200 950  1300 950
 $EndSCHEMATC
