File: doc/Boards/ConnectBoard/elec/ConnectBoard/_autosave-ConnectBoard.kicad_pcb (KiCad board)
At the start: 2 copper layers, 20 parts

Commit message: WIP
Parts:
- PropEdgeConnect-Conn1, PropEdgeConnect-Conn2, PropEdgeConnect-Conn3: moved to F.Cu
- moved PropEdgeConnect-Conn1 94.3 mm to (150.6, 100.5), turned to 0 degrees
- moved R1 49.3 mm to (52.6, 108.1)
- moved PropEdgeConnect-Conn3 46.3 mm to (70.2, 91.1), turned to 0 degrees
- moved S3 45.3 mm to (99.5, 91.1)
- moved S1 43.2 mm to (85.6, 100.8)
- moved R6 42.1 mm to (74.1, 94.8)
- moved R8 41.9 mm to (74.1, 90.8)
- moved R5 36.8 mm to (52.6, 116.2)
- moved PropEdgeConnect-Conn2 31.8 mm to (63.0, 91.1), turned to 0 degrees
- moved R7 30.3 mm to (63.4, 108.1)
- moved S5 29.6 mm to (74.9, 103.2)
- moved S7 26.9 mm to (85.6, 91.1)
- moved S0 25.0 mm to (79.5, 103.2)
- moved PS0 24.7 mm to (94.9, 91.1)
- moved S6 24.3 mm to (90.2, 91.1)
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Other:
- board outline added: 50.8 x 101.6 mm
- board text added: "For Personal Use Only."
- board text added: "SOLIDWORKS Maker Product."

Commit message: Updates
Parts:
- removed PS0: PowerSelect, Connector_PinHeader_2.54mm:PinHeader_1x03_P2.54mm_Vertical
- removed PropEdgeConnect-Conn1: PropEdgeConnect-Conn1, Connector_PinSocket_2.54mm:PinSocket_2x06_P2.54mm_Vertical
- removed PropEdgeConnect-Conn2: PropEdgeConnect-Conn2, Connector_PinSocket_2.54mm:PinSocket_2x06_P2.54mm_Vertical
- removed PropEdgeConnect-Conn3: PropEdgeConnect-Conn3, Connector_PinSocket_2.54mm:PinSocket_2x06_P2.54mm_Vertical
- removed S0: SonarConnect, Connector_PinHeader_2.54mm:PinHeader_1x03_P2.54mm_Vertical
- added Conn1: PropEdgeConnect, Connector_PinSocket_2.54mm:PinSocket_2x06_P2.54mm_Vertical, B.Cu at (177.9, 61.5)
- added Conn2: PropEdgeConnect, Connector_PinSocket_2.54mm:PinSocket_2x06_P2.54mm_Vertical, B.Cu at (198.5, 61.5)
- added Conn3: PropEdgeConnect, Connector_PinSocket_2.54mm:PinSocket_2x06_P2.54mm_Vertical, B.Cu at (199.0, 89.5)
- added Conn4: PropEdgeConnect, Connector_PinSocket_2.54mm:PinSocket_2x06_P2.54mm_Vertical, B.Cu at (200.9, 117.3)
- added J1: Prop_CommPort, Connector_PinSocket_2.54mm:PinSocket_1x04_P2.54mm_Vertical, F.Cu at (169.6, 64.0)
- added PS1: PowerSelect, Connector_PinHeader_2.54mm:PinHeader_1x03_P2.54mm_Vertical, F.Cu at (134.7, 127.2)
- added PS2: PowerSelect, Connector_PinHeader_2.54mm:PinHeader_1x03_P2.54mm_Vertical, F.Cu at (144.3, 117.5)
- added PS3: PowerSelect, Connector_PinHeader_2.54mm:PinHeader_1x03_P2.54mm_Vertical, F.Cu at (220.8, 84.0)
- added R10: 4.7k, Resistor_THT:R_Axial_DIN0207_L6.3mm_D2.5mm_P7.62mm_Horizontal, F.Cu at (84.5, 132.9)
- added R11: 4.7k, Resistor_THT:R_Axial_DIN0207_L6.3mm_D2.5mm_P7.62mm_Horizontal, F.Cu at (84.5, 137.0)
- added R12: 4.7k, Resistor_THT:R_Axial_DIN0207_L6.3mm_D2.5mm_P7.62mm_Horizontal, F.Cu at (114.2, 107.5)
- added R13: 4.7k, Resistor_THT:R_Axial_DIN0207_L6.3mm_D2.5mm_P7.62mm_Horizontal, F.Cu at (211.2, 56.2)
- added R14: 4.7k, Resistor_THT:R_Axial_DIN0207_L6.3mm_D2.5mm_P7.62mm_Horizontal, F.Cu at (211.2, 62.2)
- added R15: 4.7k, Resistor_THT:R_Axial_DIN0207_L6.3mm_D2.5mm_P7.62mm_Horizontal, F.Cu at (211.2, 68.2)
- added R16: 4.7k, Resistor_THT:R_Axial_DIN0207_L6.3mm_D2.5mm_P7.62mm_Horizontal, F.Cu at (211.2, 74.2)
- added R17: 4.7k, Resistor_THT:R_Axial_DIN0207_L6.3mm_D2.5mm_P7.62mm_Horizontal, F.Cu at (95.3, 132.9)
- added R18: 4.7k, Resistor_THT:R_Axial_DIN0207_L6.3mm_D2.5mm_P7.62mm_Horizontal, F.Cu at (109.6, 119.7)
- added R19: 4.7k, Resistor_THT:R_Axial_DIN0207_L6.3mm_D2.5mm_P7.62mm_Horizontal, F.Cu at (88.2, 145.1)
- added R20: 4.7k, Resistor_THT:R_Axial_DIN0207_L6.3mm_D2.5mm_P7.62mm_Horizontal, F.Cu at (109.6, 123.8)
- added R21: 4.7k, Resistor_THT:R_Axial_DIN0207_L6.3mm_D2.5mm_P7.62mm_Horizontal, F.Cu at (211.2, 59.2)
- added R22: 4.7k, Resistor_THT:R_Axial_DIN0207_L6.3mm_D2.5mm_P7.62mm_Horizontal, F.Cu at (211.2, 65.2)
- added R23: 4.7k, Resistor_THT:R_Axial_DIN0207_L6.3mm_D2.5mm_P7.62mm_Horizontal, F.Cu at (211.2, 71.2)
- added R24: 4.7k, Resistor_THT:R_Axial_DIN0207_L6.3mm_D2.5mm_P7.62mm_Horizontal, F.Cu at (211.2, 77.2)
- added R9: 4.7k, Resistor_THT:R_Axial_DIN0207_L6.3mm_D2.5mm_P7.62mm_Horizontal, F.Cu at (77.4, 142.2)
- added S10: SonarConnect, Connector_PinHeader_2.54mm:PinHeader_1x03_P2.54mm_Vertical, F.Cu at (115.1, 137.8)
- added S11: SonarConnect, Connector_PinHeader_2.54mm:PinHeader_1x03_P2.54mm_Vertical, F.Cu at (146.2, 150.5)
- added S12: SonarConnect, Connector_PinHeader_2.54mm:PinHeader_1x03_P2.54mm_Vertical, F.Cu at (145.8, 107.8)
- added S13: SonarConnect, Connector_PinHeader_2.54mm:PinHeader_1x03_P2.54mm_Vertical, F.Cu at (106.8, 128.1)
- added S14: SonarConnect, Connector_PinHeader_2.54mm:PinHeader_1x03_P2.54mm_Vertical, F.Cu at (139.7, 117.5)
- added S15: SonarConnect, Connector_PinHeader_2.54mm:PinHeader_1x03_P2.54mm_Vertical, F.Cu at (115.0, 156.0)
- added S16: SonarConnect, Connector_PinHeader_2.54mm:PinHeader_1x03_P2.54mm_Vertical, F.Cu at (231.9, 74.4)
- added S17: SonarConnect, Connector_PinHeader_2.54mm:PinHeader_1x03_P2.54mm_Vertical, F.Cu at (150.5, 107.8)
- added S18: SonarConnect, Connector_PinHeader_2.54mm:PinHeader_1x03_P2.54mm_Vertical, F.Cu at (139.4, 127.2)
- added S19: SonarConnect, Connector_PinHeader_2.54mm:PinHeader_1x03_P2.54mm_Vertical, F.Cu at (149.0, 117.5)
- added S20: SonarConnect, Connector_PinHeader_2.54mm:PinHeader_1x03_P2.54mm_Vertical, F.Cu at (126.9, 156.8)
- added S21: SonarConnect, Connector_PinHeader_2.54mm:PinHeader_1x03_P2.54mm_Vertical, F.Cu at (144.0, 127.2)
- added S22: SonarConnect, Connector_PinHeader_2.54mm:PinHeader_1x03_P2.54mm_Vertical, F.Cu at (135.0, 117.5)
- added S23: SonarConnect, Connector_PinHeader_2.54mm:PinHeader_1x03_P2.54mm_Vertical, F.Cu at (231.9, 71.9)
- added S24: SonarConnect, Connector_PinHeader_2.54mm:PinHeader_1x03_P2.54mm_Vertical, F.Cu at (231.9, 77.0)
- added S8: SonarConnect, Connector_PinHeader_2.54mm:PinHeader_1x03_P2.54mm_Vertical, F.Cu at (130.4, 116.0)
- added S9: SonarConnect, Connector_PinHeader_2.54mm:PinHeader_1x03_P2.54mm_Vertical, F.Cu at (125.4, 125.7)
- moved R5 158.3 mm to (209.0, 92.0)
- moved R6 152.4 mm to (226.5, 94.5), turned to 180 degrees
- moved S6 53.6 mm to (141.2, 107.8)
- moved S7 51.1 mm to (120.8, 128.1)
- moved R1 50.8 mm to (103.5, 107.5)
- moved S5 49.6 mm to (110.5, 137.8)
- moved R2 46.9 mm to (98.8, 119.8)
- moved S4 42.2 mm to (136.5, 107.8)
- moved R7 40.8 mm to (103.5, 115.7)
- moved S3 40.6 mm to (116.1, 128.1)
- moved R8 39.5 mm to (84.5, 128.9)
- moved S2 38.6 mm to (125.7, 116.0)
- moved S1 37.7 mm to (111.5, 128.1)
- moved R3 32.0 mm to (103.5, 111.6)
- moved R4 24.7 mm to (84.5, 124.8)
Connections:
- R1 pad 1: /P0 -> /P55
- R2 pad 1: /P2 -> /P53
- R3 pad 1: /P4 -> /P51
- R4 pad 1: /P6 -> /P49
- R5 pad 2: /P1 -> /P54
- R6 pad 2: /P3 -> /P52
- R7 pad 2: /P5 -> /P50
- R8 pad 2: /P7 -> /P48
- S1 pad 1: Net-(R5-Pad1) -> Net-(R1-Pad2)
- S3 pad 1: Net-(R6-Pad1) -> Net-(R3-Pad2)
- S4 pad 1: Net-(R3-Pad2) -> Net-(R4-Pad2)
- S5 pad 1: Net-(R7-Pad1) -> Net-(R5-Pad1)
- S6 pad 1: Net-(R4-Pad2) -> Net-(R6-Pad1)
- S7 pad 1: Net-(R8-Pad1) -> Net-(R7-Pad1)
