File: doc/Boards/ConnectBoard/elec/ConnectBoard/ConnectBoard.kicad_pcb (KiCad board)
At the start: 2 copper layers, 4 parts, among them J1 Sonar0, J2 PowerSelect0, J3 PropEdgeConnect-Conn1

Commit message: WIP
Parts:
- added PropEdgeConnect-Conn2: PropEdgeConnect-Conn2, Connector_PinSocket_2.54mm:PinSocket_2x06_P2.54mm_Vertical, B.Cu at (78.0, 63.0)
- added PropEdgeConnect-Conn3: PropEdgeConnect-Conn3, Connector_PinSocket_2.54mm:PinSocket_2x06_P2.54mm_Vertical, B.Cu at (107.0, 63.0)
- added R2: 4.7k, Resistor_THT:R_Axial_DIN0207_L6.3mm_D2.5mm_P7.62mm_Horizontal, F.Cu at (67.0, 110.0)
- added R3: 4.7k, Resistor_THT:R_Axial_DIN0207_L6.3mm_D2.5mm_P7.62mm_Horizontal, F.Cu at (67.0, 114.0)
- added R4: 4.7k, Resistor_THT:R_Axial_DIN0207_L6.3mm_D2.5mm_P7.62mm_Horizontal, F.Cu at (77.8, 110.0)
- added S1: S0, Connector_PinHeader_2.54mm:PinHeader_1x03_P2.54mm_Vertical, F.Cu at (78.5, 114.3)
- added S2: S0, Connector_PinHeader_2.54mm:PinHeader_1x03_P2.54mm_Vertical, F.Cu at (89.3, 110.3)
- added S3: S0, Connector_PinHeader_2.54mm:PinHeader_1x03_P2.54mm_Vertical, F.Cu at (83.2, 114.3)
- S0: renamed from J1; value Sonar0 -> S0
- moved PropEdgeConnect-Conn1 40.2 mm to (64.0, 63.0), turned to 90 degrees
- renumbered J2 to PowerSelect0, J3 to PropEdgeConnect-Conn1
Connections:
- PropEdgeConnect-Conn1 pad 3: Net-(J3-Pad3) -> /P2
- PropEdgeConnect-Conn1 pad 4: Net-(J3-Pad4) -> /P4
- PropEdgeConnect-Conn1 pad 5: Net-(J3-Pad5) -> /P6

Commit message: WIP
Parts:
- added R5: 4.7k, Resistor_THT:R_Axial_DIN0207_L6.3mm_D2.5mm_P7.62mm_Horizontal, F.Cu at (32.3, 85.5)
- added R6: 4.7k, Resistor_THT:R_Axial_DIN0207_L6.3mm_D2.5mm_P7.62mm_Horizontal, F.Cu at (32.3, 89.6)
- added R7: 4.7k, Resistor_THT:R_Axial_DIN0207_L6.3mm_D2.5mm_P7.62mm_Horizontal, F.Cu at (43.0, 85.5)
- added R8: 4.7k, Resistor_THT:R_Axial_DIN0207_L6.3mm_D2.5mm_P7.62mm_Horizontal, F.Cu at (32.3, 93.7)
- added S1: SonarConnect, Connector_PinHeader_2.54mm:PinHeader_1x03_P2.54mm_Vertical, F.Cu at (43.8, 89.9)
- added S3: SonarConnect, Connector_PinHeader_2.54mm:PinHeader_1x03_P2.54mm_Vertical, F.Cu at (54.6, 85.8)
- added S5: SonarConnect, Connector_PinHeader_2.54mm:PinHeader_1x03_P2.54mm_Vertical, F.Cu at (48.4, 89.9)
- added S7: SonarConnect, Connector_PinHeader_2.54mm:PinHeader_1x03_P2.54mm_Vertical, F.Cu at (59.2, 85.8)
- PS0: renamed from PowerSelect0; value PowerSelect0 -> PowerSelect
- S0: value S0 -> SonarConnect
- S2: renamed from S1; value S0 -> SonarConnect
- S4: renamed from S2; value S0 -> SonarConnect
- S6: renamed from S3; value S0 -> SonarConnect
Connections:
- PropEdgeConnect-Conn1 pad 10: Net-(PropEdgeConnect-Conn1-Pad10) -> /P5
- PropEdgeConnect-Conn1 pad 11: Net-(PropEdgeConnect-Conn1-Pad11) -> /P7
- PropEdgeConnect-Conn1 pad 8: Net-(PropEdgeConnect-Conn1-Pad8) -> /P1
- PropEdgeConnect-Conn1 pad 9: Net-(PropEdgeConnect-Conn1-Pad9) -> /P3
Other:
- board outline added: 50.8 x 101.6 mm
- board text added: "For Personal Use Only."
- board text added: "SOLIDWORKS Maker Product."

Commit message: Updates
Parts:
- removed PS0: PowerSelect, Connector_PinHeader_2.54mm:PinHeader_1x03_P2.54mm_Vertical
- removed PropEdgeConnect-Conn1: PropEdgeConnect-Conn1, Connector_PinSocket_2.54mm:PinSocket_2x06_P2.54mm_Vertical
- removed PropEdgeConnect-Conn2: PropEdgeConnect-Conn2, Connector_PinSocket_2.54mm:PinSocket_2x06_P2.54mm_Vertical
- removed PropEdgeConnect-Conn3: PropEdgeConnect-Conn3, Connector_PinSocket_2.54mm:PinSocket_2x06_P2.54mm_Vertical
- removed S0: SonarConnect, Connector_PinHeader_2.54mm:PinHeader_1x03_P2.54mm_Vertical
- added Conn1: PropEdgeConnect, Connector_PinSocket_2.54mm:PinSocket_2x06_P2.54mm_Vertical, B.Cu at (177.9, 61.5)
- added Conn2: PropEdgeConnect, Connector_PinSocket_2.54mm:PinSocket_2x06_P2.54mm_Vertical, B.Cu at (198.5, 61.5)
- added Conn3: PropEdgeConnect, Connector_PinSocket_2.54mm:PinSocket_2x06_P2.54mm_Vertical, B.Cu at (199.0, 89.5)
- added Conn4: PropEdgeConnect, Connector_PinSocket_2.54mm:PinSocket_2x06_P2.54mm_Vertical, B.Cu at (200.9, 117.3)
- added J1: Prop_CommPort, Connector_PinSocket_2.54mm:PinSocket_1x04_P2.54mm_Vertical, F.Cu at (169.6, 64.0)
- added PS1: PowerSelect, Connector_PinHeader_2.54mm:PinHeader_1x03_P2.54mm_Vertical, F.Cu at (134.7, 127.2)
- added PS2: PowerSelect, Connector_PinHeader_2.54mm:PinHeader_1x03_P2.54mm_Vertical, F.Cu at (144.3, 117.5)
- added PS3: PowerSelect, Connector_PinHeader_2.54mm:PinHeader_1x03_P2.54mm_Vertical, F.Cu at (125.4, 135.3)
- added R10: 4.7k, Resistor_THT:R_Axial_DIN0207_L6.3mm_D2.5mm_P7.62mm_Horizontal, F.Cu at (84.5, 132.9)
- added R11: 4.7k, Resistor_THT:R_Axial_DIN0207_L6.3mm_D2.5mm_P7.62mm_Horizontal, F.Cu at (84.5, 137.0)
- added R12: 4.7k, Resistor_THT:R_Axial_DIN0207_L6.3mm_D2.5mm_P7.62mm_Horizontal, F.Cu at (114.2, 107.5)
- added R13: 4.7k, Resistor_THT:R_Axial_DIN0207_L6.3mm_D2.5mm_P7.62mm_Horizontal, F.Cu at (221.0, 52.0)
- added R14: 4.7k, Resistor_THT:R_Axial_DIN0207_L6.3mm_D2.5mm_P7.62mm_Horizontal, F.Cu at (221.0, 61.0)
- added R15: 4.7k, Resistor_THT:R_Axial_DIN0207_L6.3mm_D2.5mm_P7.62mm_Horizontal, F.Cu at (221.5, 69.0)
- added R16: 4.7k, Resistor_THT:R_Axial_DIN0207_L6.3mm_D2.5mm_P7.62mm_Horizontal, F.Cu at (220.5, 76.5)
- added R17: 4.7k, Resistor_THT:R_Axial_DIN0207_L6.3mm_D2.5mm_P7.62mm_Horizontal, F.Cu at (95.3, 132.9)
- added R18: 4.7k, Resistor_THT:R_Axial_DIN0207_L6.3mm_D2.5mm_P7.62mm_Horizontal, F.Cu at (109.6, 119.7)
- added R19: 4.7k, Resistor_THT:R_Axial_DIN0207_L6.3mm_D2.5mm_P7.62mm_Horizontal, F.Cu at (88.2, 145.1)
- added R20: 4.7k, Resistor_THT:R_Axial_DIN0207_L6.3mm_D2.5mm_P7.62mm_Horizontal, F.Cu at (109.6, 123.8)
- added R21: 4.7k, Resistor_THT:R_Axial_DIN0207_L6.3mm_D2.5mm_P7.62mm_Horizontal, F.Cu at (228.5, 56.0)
- added R22: 4.7k, Resistor_THT:R_Axial_DIN0207_L6.3mm_D2.5mm_P7.62mm_Horizontal, F.Cu at (229.0, 65.0)
- added R23: 4.7k, Resistor_THT:R_Axial_DIN0207_L6.3mm_D2.5mm_P7.62mm_Horizontal, F.Cu at (228.5, 72.5)
- added R24: 4.7k, Resistor_THT:R_Axial_DIN0207_L6.3mm_D2.5mm_P7.62mm_Horizontal, F.Cu at (229.5, 84.0)
- added R9: 4.7k, Resistor_THT:R_Axial_DIN0207_L6.3mm_D2.5mm_P7.62mm_Horizontal, F.Cu at (77.4, 142.2)
- added S10: SonarConnect, Connector_PinHeader_2.54mm:PinHeader_1x03_P2.54mm_Vertical, F.Cu at (115.1, 137.8)
- added S11: SonarConnect, Connector_PinHeader_2.54mm:PinHeader_1x03_P2.54mm_Vertical, F.Cu at (146.2, 150.5)
- added S12: SonarConnect, Connector_PinHeader_2.54mm:PinHeader_1x03_P2.54mm_Vertical, F.Cu at (145.8, 107.8)
- added S13: SonarConnect, Connector_PinHeader_2.54mm:PinHeader_1x03_P2.54mm_Vertical, F.Cu at (106.8, 128.1)
- added S14: SonarConnect, Connector_PinHeader_2.54mm:PinHeader_1x03_P2.54mm_Vertical, F.Cu at (139.7, 117.5)
- added S15: SonarConnect, Connector_PinHeader_2.54mm:PinHeader_1x03_P2.54mm_Vertical, F.Cu at (115.0, 156.0)
- added S16: SonarConnect, Connector_PinHeader_2.54mm:PinHeader_1x03_P2.54mm_Vertical, F.Cu at (130.1, 125.7)
- added S17: SonarConnect, Connector_PinHeader_2.54mm:PinHeader_1x03_P2.54mm_Vertical, F.Cu at (150.5, 107.8)
- added S18: SonarConnect, Connector_PinHeader_2.54mm:PinHeader_1x03_P2.54mm_Vertical, F.Cu at (139.4, 127.2)
- added S19: SonarConnect, Connector_PinHeader_2.54mm:PinHeader_1x03_P2.54mm_Vertical, F.Cu at (149.0, 117.5)
- added S20: SonarConnect, Connector_PinHeader_2.54mm:PinHeader_1x03_P2.54mm_Vertical, F.Cu at (126.9, 156.8)
- added S21: SonarConnect, Connector_PinHeader_2.54mm:PinHeader_1x03_P2.54mm_Vertical, F.Cu at (144.0, 127.2)
- added S22: SonarConnect, Connector_PinHeader_2.54mm:PinHeader_1x03_P2.54mm_Vertical, F.Cu at (135.0, 117.5)
- added S23: SonarConnect, Connector_PinHeader_2.54mm:PinHeader_1x03_P2.54mm_Vertical, F.Cu at (253.5, 120.0)
- added S24: SonarConnect, Connector_PinHeader_2.54mm:PinHeader_1x03_P2.54mm_Vertical, F.Cu at (244.5, 76.5)
- added S8: SonarConnect, Connector_PinHeader_2.54mm:PinHeader_1x03_P2.54mm_Vertical, F.Cu at (130.4, 116.0)
- added S9: SonarConnect, Connector_PinHeader_2.54mm:PinHeader_1x03_P2.54mm_Vertical, F.Cu at (125.4, 125.7)
- moved R6 194.3 mm to (226.5, 94.5), turned to 180 degrees
- moved R5 176.8 mm to (209.0, 92.0)
- moved S5 78.4 mm to (110.5, 137.8)
- moved S1 77.7 mm to (111.5, 128.1)
- moved S3 74.7 mm to (116.1, 128.1)
- moved S7 74.7 mm to (120.8, 128.1)
- moved R7 67.5 mm to (103.5, 115.7)
- moved R8 63.1 mm to (84.5, 128.9)
- moved S6 58.4 mm to (141.2, 107.8)
- moved S4 47.3 mm to (136.5, 107.8)
- moved S2 47.2 mm to (125.7, 116.0)
- moved R3 36.5 mm to (103.5, 111.6)
- moved R2 33.3 mm to (98.8, 119.8)
- moved R1 26.0 mm to (103.5, 107.5)
- moved R4 16.3 mm to (84.5, 124.8)
Connections:
- R1 pad 1: /P0 -> /P55
- R2 pad 1: /P2 -> /P53
- R3 pad 1: /P4 -> /P51
- R4 pad 1: /P6 -> /P49
- R5 pad 2: /P1 -> /P54
- R6 pad 2: /P3 -> /P52
- R7 pad 2: /P5 -> /P50
- R8 pad 2: /P7 -> /P48
- S1 pad 1: Net-(R5-Pad1) -> Net-(R1-Pad2)
- S3 pad 1: Net-(R6-Pad1) -> Net-(R3-Pad2)
- S4 pad 1: Net-(R3-Pad2) -> Net-(R4-Pad2)
- S5 pad 1: Net-(R7-Pad1) -> Net-(R5-Pad1)
- S6 pad 1: Net-(R4-Pad2) -> Net-(R6-Pad1)
- S7 pad 1: Net-(R8-Pad1) -> Net-(R7-Pad1)
Other:
- outline, holes or cut-outs redrawn

Commit message: More work on this.
Parts:
- removed R10, R11, R12, R13, R14, R15, R16, R17, R18, R19, R20, R21, R22, R23, R24, R7, R8, R9: 4.7k, Resistor_THT:R_Axial_DIN0207_L6.3mm_D2.5mm_P7.62mm_Horizontal
- J0: renamed from J1; footprint Connector_PinSocket_2.54mm:PinSocket_1x04_P2.54mm_Vertical -> Connector_PinHeader_2.54mm:PinHeader_1x04_P2.54mm_Vertical
- R1, R2: footprint Resistor_THT:R_Axial_DIN0207_L6.3mm_D2.5mm_P7.62mm_Horizontal -> Package_DIP:DIP-8_W7.62mm
- R3, R4, R5, R6: value 4.7k -> R_Pack04_Split; footprint Resistor_THT:R_Axial_DIN0207_L6.3mm_D2.5mm_P7.62mm_Horizontal -> Package_DIP:DIP-8_W7.62mm
- moved S24 158.5 mm to (93.9, 126.0), turned to 0 degrees
- moved R4 134.0 mm to (217.2, 105.4)
- moved S5 129.1 mm to (220.0, 69.3), turned to 90 degrees
- moved S23 119.7 mm to (135.1, 102.5)
- moved R2 119.2 mm to (208.0, 71.9)
- moved S1 118.9 mm to (220.0, 79.5), turned to 90 degrees
- moved S7 117.9 mm to (220.0, 64.3), turned to 90 degrees
- moved S3 116.9 mm to (220.0, 74.4), turned to 90 degrees
- moved R3 115.6 mm to (217.7, 93.7)
- moved R1 114.2 mm to (208.0, 61.7)
- moved S8 104.7 mm to (220.0, 61.7), turned to 90 degrees
- moved S2 102.0 mm to (220.0, 77.0), turned to 90 degrees
- moved PS1 95.0 mm to (220.0, 85.3), turned to 90 degrees
- moved S4 90.9 mm to (220.0, 71.9), turned to 90 degrees
- moved S6 88.9 mm to (220.0, 66.8), turned to 90 degrees
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Connections:
- PS1 pad 1: V48 -> V56
- PS2 pad 1: V40 -> V48
- PS2 pad 3: +5V3 -> +5V1
- PS3 pad 1: V56 -> V40
- PS3 pad 3: +5V1 -> +5V3
- R1 pad 1: /P55 -> /P63
- R1 pad 2: Net-(R1-Pad2) -> /P62
- R2 pad 1: /P53 -> /P59
- R2 pad 2: Net-(R2-Pad2) -> /P58
- R3 pad 1: /P51 -> Net-(R3-Pad1)
- R4 pad 1: /P49 -> /P54
- R4 pad 2: Net-(R4-Pad2) -> /P52
- R5 pad 2: /P54 -> Net-(R5-Pad2)
- R6 pad 1: Net-(R6-Pad1) -> /P46
- R6 pad 2: /P52 -> /P44
- S1 pad 1: Net-(R1-Pad2) -> Net-(R2-Pad5)
- S10 pad 1: Net-(R10-Pad2) -> Net-(R3-Pad4)
- S11 pad 1: Net-(R11-Pad2) -> Net-(R4-Pad6)
- S12 pad 1: Net-(R12-Pad2) -> Net-(R3-Pad3)
- S13 pad 1: Net-(R13-Pad2) -> Net-(R4-Pad7)
- S13 pad 2: Net-(PS3-Pad2) -> Net-(PS2-Pad2)
- S14 pad 1: Net-(R14-Pad2) -> Net-(R3-Pad2)
- S14 pad 2: Net-(PS3-Pad2) -> Net-(PS2-Pad2)
- S15 pad 1: Net-(R15-Pad2) -> Net-(R4-Pad8)
- S15 pad 2: Net-(PS3-Pad2) -> Net-(PS2-Pad2)
- S16 pad 1: Net-(R16-Pad2) -> Net-(R3-Pad1)
- S16 pad 2: Net-(PS3-Pad2) -> Net-(PS2-Pad2)
- S17 pad 1: Net-(R17-Pad1) -> Net-(R6-Pad5)
- S17 pad 2: Net-(PS2-Pad2) -> Net-(PS3-Pad2)
- S18 pad 1: Net-(R18-Pad1) -> Net-(R5-Pad4)
- S18 pad 2: Net-(PS2-Pad2) -> Net-(PS3-Pad2)
- S19 pad 1: Net-(R19-Pad1) -> Net-(R6-Pad6)
- S19 pad 2: Net-(PS2-Pad2) -> Net-(PS3-Pad2)
- S2 pad 1: Net-(R2-Pad2) -> Net-(R2-Pad6)
- S20 pad 1: Net-(R20-Pad1) -> Net-(R5-Pad3)
- S20 pad 2: Net-(PS2-Pad2) -> Net-(PS3-Pad2)
- S21 pad 1: Net-(R21-Pad1) -> Net-(R6-Pad7)
- S22 pad 1: Net-(R22-Pad1) -> Net-(R5-Pad2)
- S23 pad 1: Net-(R23-Pad1) -> Net-(R6-Pad8)
- S24 pad 1: Net-(R24-Pad1) -> Net-(R5-Pad1)
- S3 pad 1: Net-(R3-Pad2) -> Net-(R2-Pad7)
- S4 pad 1: Net-(R4-Pad2) -> Net-(R2-Pad8)
- S5 pad 1: Net-(R5-Pad1) -> Net-(R1-Pad5)
- S6 pad 1: Net-(R6-Pad1) -> Net-(R1-Pad6)
- S7 pad 1: Net-(R7-Pad1) -> Net-(R1-Pad7)
- S8 pad 1: Net-(R8-Pad1) -> Net-(R1-Pad8)
- S9 pad 1: Net-(R9-Pad2) -> Net-(R4-Pad5)
Routing:
- net GND: track 0.00 -> 49.2 mm
- net V56: track 0.00 -> 41.4 mm
- net Net-(PS1-Pad2): track 0.00 -> 23.6 mm
- net /P57: track 0.00 -> 12.8 mm
- net /P59: track 0.00 -> 11.7 mm
- net /P56: track 0.00 -> 10.8 mm
- net /P61: track 0.00 -> 10.6 mm
- net /P63: track 0.00 -> 10.5 mm
- net /P58: track 0.00 -> 9.20 mm
- net /P60: track 0.00 -> 8.16 mm
- net /P62: track 0.00 -> 7.09 mm
- net Net-(R2-Pad8): track 0.00 -> 4.32 mm
- net Net-(R2-Pad7): track 0.00 -> 4.32 mm
- net Net-(R2-Pad6): track 0.00 -> 4.32 mm
- net Net-(R2-Pad5): track 0.00 -> 4.32 mm
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Other:
- board size 50.8 x 101.6 mm -> 63.5 x 82.9 mm

Commit message: Updates
Parts:
- moved R5 85.2 mm to (138.7, 117.4)
- moved R6 84.6 mm to (138.7, 106.7)
- moved R4 82.6 mm to (138.7, 79.5)
- moved R3 79.1 mm to (138.7, 89.7)
- moved Conn4 71.4 mm to (130.0, 108.6)
- moved Conn1 71.3 mm to (107.2, 52.7)
- moved J0 70.6 mm to (99.1, 60.7), turned to 180 degrees
- moved PS1 69.9 mm to (150.8, 75.2)
- moved R1 69.7 mm to (138.9, 53.1)
- moved R2 69.7 mm to (138.9, 63.3)
- moved S1 69.7 mm to (150.8, 70.9)
- moved S2 69.7 mm to (150.8, 68.4)
- moved S3 69.7 mm to (150.8, 65.9)
- moved S4 69.7 mm to (150.8, 63.3)
- moved S5 69.7 mm to (150.8, 60.8)
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Connections:
- R3 pad 1: Net-(R3-Pad1) -> /P51
- R3 pad 2: Net-(R3-Pad2) -> /P50
- R3 pad 3: Net-(R3-Pad3) -> /P49
- R3 pad 4: Net-(R3-Pad4) -> /P48
- R3 pad 5: /P49 -> Net-(R3-Pad5)
- R3 pad 6: /P51 -> Net-(R3-Pad6)
- R3 pad 7: /P53 -> Net-(R3-Pad7)
- R3 pad 8: /P55 -> Net-(R3-Pad8)
- R4 pad 1: /P54 -> /P55
- R4 pad 2: /P52 -> /P54
- R4 pad 3: /P50 -> /P53
- R4 pad 4: /P48 -> /P52
- R5 pad 1: Net-(R5-Pad1) -> /P43
- R5 pad 2: Net-(R5-Pad2) -> /P42
- R5 pad 3: Net-(R5-Pad3) -> /P41
- R5 pad 4: Net-(R5-Pad4) -> /P40
- R5 pad 5: /P41 -> Net-(R5-Pad5)
- R5 pad 6: /P43 -> Net-(R5-Pad6)
- R5 pad 7: /P45 -> Net-(R5-Pad7)
- R5 pad 8: /P47 -> Net-(R5-Pad8)
- R6 pad 1: /P46 -> /P47
- R6 pad 2: /P44 -> /P46
- R6 pad 3: /P42 -> /P45
- R6 pad 4: /P40 -> /P44
- S10 pad 1: Net-(R3-Pad4) -> Net-(R3-Pad6)
- S11 pad 1: Net-(R4-Pad6) -> Net-(R3-Pad7)
- S12 pad 1: Net-(R3-Pad3) -> Net-(R3-Pad8)
- S13 pad 1: Net-(R4-Pad7) -> Net-(R4-Pad5)
- S14 pad 1: Net-(R3-Pad2) -> Net-(R4-Pad6)
- S15 pad 1: Net-(R4-Pad8) -> Net-(R4-Pad7)
- S16 pad 1: Net-(R3-Pad1) -> Net-(R4-Pad8)
- S17 pad 1: Net-(R6-Pad5) -> Net-(R5-Pad5)
- S18 pad 1: Net-(R5-Pad4) -> Net-(R5-Pad6)
- S19 pad 1: Net-(R6-Pad6) -> Net-(R5-Pad7)
- S20 pad 1: Net-(R5-Pad3) -> Net-(R5-Pad8)
- S21 pad 1: Net-(R6-Pad7) -> Net-(R6-Pad5)
- S22 pad 1: Net-(R5-Pad2) -> Net-(R6-Pad6)
- S23 pad 1: Net-(R6-Pad8) -> Net-(R6-Pad7)
- S24 pad 1: Net-(R5-Pad1) -> Net-(R6-Pad8)
- S9 pad 1: Net-(R4-Pad5) -> Net-(R3-Pad5)
Routing:
- net GND: track 49.2 -> 196.9 mm
- net +5V1: track 0.00 -> 81.6 mm
- net +5V3: track 0.00 -> 54.5 mm
- net V40: track 0.00 -> 40.4 mm
- net V48: track 0.00 -> 40.1 mm
- net Net-(PS3-Pad2): track 0.00 -> 22.6 mm
- net Net-(PS2-Pad2): track 0.00 -> 22.1 mm
- net /P49: track 0.00 -> 11.3 mm
- net /P41: track 0.00 -> 11.2 mm
- net /P43: track 0.00 -> 10.7 mm
- net /P47: track 0.00 -> 10.5 mm
- net /P0: track 0.00 -> 10.4 mm
- net /P51: track 0.00 -> 10.2 mm
- net /P55: track 0.00 -> 10.2 mm
- net /P45: track 0.00 -> 9.45 mm
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Other:
- outline, holes or cut-outs redrawn
- board text removed: "For Personal Use Only."
- board text removed: "SOLIDWORKS Maker Product."

Commit message: WIP
Parts:
- moved R5 0.51 mm to (138.7, 116.8)
- moved S17 0.51 mm to (150.9, 124.5)
- moved S18 0.51 mm to (150.9, 121.9)
- moved S19 0.51 mm to (150.9, 119.4)
- moved S20 0.51 mm to (150.9, 116.8)
- moved PS3 0.49 mm to (150.9, 128.8)
Routing:
- net GND: track 196.9 -> 195.6 mm, vias 0 -> 1
- net /P41: track 11.2 -> 12.1 mm
- net V40: track 40.4 -> 41.3 mm

Commit message: WIP
Parts:
- J0: value Prop_CommPort -> Comm Port
- moved J0 5.71 mm to (100.4, 55.1), turned to 0 degrees
Connections:
- J0 pad 1: /P0 -> GND
- J0 pad 2: /P2 -> Net-(J0-Pad2)
- J0 pad 3: Net-(J0-Pad3) -> /P0
- J0 pad 4: GND -> /P2
Routing:
- net /P0: track 10.4 -> 8.87 mm
- net /P2: track 8.26 -> 9.41 mm
Other:
- board text added: "<TX"
- board text added: ">RX"
- board text added: "DC Jack Below"
- board text added: "M3"
- board text added: "NC"
- board text added: "Propeller 2 Edge Breakout Sonar Connect DPG 2025 Rev0"
- board text added: "Sonar1 - - -> Sonar8"
- board text added: "Sonar17 - - -> Sonar24"
- board text added: "Sonar9 - - -> Sonar16"
- board text added: "Vss"
