File: doc/Boards/ConnectBoard/elec/ConnectBoard/ConnectBoard.kicad_pcb (KiCad board)
At the start: 2 copper layers, 63.5 x 82.9 mm, 38 parts, among them J0 Comm Port

Commit message: Updates
Other:
- board text added: "3.3V"
- board text added: "5V"
- board text added: "S + -"
Changed lines of the file:
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@@
   (general
     (thickness 1.6)
-    (drawings 22)
+    (drawings 25)
     (tracks 254)
     (zones 0)
@@
     )
   )
+  (gr_text "S + -" (at 153.5504 73.1504) (layer F.Cu)
+    (effects (font (size 1.35 1.35) (thickness 0.3)))
+  )
+  (gr_text 5V (at 156.2354 77.4954) (layer F.Cu)
+    (effects (font (size 1 1) (thickness 0.25)))
+  )
+  (gr_text 3.3V (at 149.8854 77.4954) (layer F.Cu)
+    (effects (font (size 1 1) (thickness 0.25)))
+  )
   (gr_text M3 (at 128.0414 130.8354) (layer F.SilkS)

Commit message: Work Complete
Other:
- board text added: "P0"
- board text added: "P2"
- board text added: "P40"
- board text added: "P41"
- board text added: "P42"
- board text added: "P43"
- board text added: "P44"
- board text added: "P45"
- board text added: "P46"
- board text added: "P47"
- board text added: "P48"
- board text added: "P49"
- board text added: "P50"
- board text added: "P51"
- board text added: "P52"
- board text added: "P53"
- board text added: "P54"
- board text added: "P55"
- board text added: "P56"
- board text added: "P57"
- board text added: "P58"
- board text added: "P59"
- board text added: "P60"
- board text added: "P61"
- board text added: "P62"
- board text added: "P63"
- board text added: "Propeller 2 Edge Breakout Sonar Connect DPG 2025 Rev1"
- board text removed: "Propeller 2 Edge Breakout Sonar Connect DPG 2025 Rev0"
Changed lines of the file:
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@@
   (general
     (thickness 1.6)
-    (drawings 25)
+    (drawings 57)
     (tracks 254)
     (zones 0)
@@
   (title_block
     (title "Prop 2 Sonar Connect Board")
-    (date 2025-03-25)
-    (rev Rev0)
+    (date 2025-04-08)
+    (rev Rev1)
     (company "FAST Robotics")
   )
@@
       (effects (font (size 1 1) (thickness 0.15)))
     )
-    (fp_text value "Comm Port" (at 2.286 3.81 270 unlocked) (layer F.SilkS)
+    (fp_text value "Comm Port" (at 0.254 -2.032 unlocked) (layer F.SilkS)
       (effects (font (size 1 1) (thickness 0.15)))
     )
@@
     )
   )
-  (gr_text "S + -" (at 153.5504 73.1504) (layer F.Cu)
-    (effects (font (size 1.35 1.35) (thickness 0.3)))
-  )
-  (gr_text 5V (at 156.2354 77.4954) (layer F.Cu)
+  (gr_text P2 (at 102.6414 62.7634) (layer F.SilkS)
+    (effects (font (size 0.8 0.8) (thickness 0.15)))
+  )
+  (gr_text P0 (at 102.6414 60.2234) (layer F.SilkS)
+    (effects (font (size 0.8 0.8) (thickness 0.15)))
+  )
+  (gr_text P40 (at 136.4234 124.7394) (layer F.SilkS)
+    (effects (font (size 0.8 0.8) (thickness 0.15)))
+  )
+  (gr_text P41 (at 136.4234 122.1994) (layer F.SilkS)
+    (effects (font (size 0.8 0.8) (thickness 0.15)))
+  )
+  (gr_text P42 (at 136.4234 119.4054) (layer F.SilkS)
+    (effects (font (size 0.8 0.8) (thickness 0.15)))
+  )
+  (gr_text P43 (at 136.4234 116.8654) (layer F.SilkS)
+    (effects (font (size 0.8 0.8) (thickness 0.15)))
+  )
+  (gr_text P44 (at 136.4234 114.5794) (layer F.SilkS)
+    (effects (font (size 0.8 0.8) (thickness 0.15)))
+  )
+  (gr_text P45 (at 136.4234 112.0394) (layer F.SilkS)
+    (effects (font (size 0.8 0.8) (thickness 0.15)))
+  )
+  (gr_text P46 (at 136.4234 109.4994) (layer F.SilkS)
+    (effects (font (size 0.8 0.8) (thickness 0.15)))
+  )
+  (gr_text P47 (at 136.4234 106.9594) (layer F.SilkS)
+    (effects (font (size 0.8 0.8) (thickness 0.15)))
+  )
+  (gr_text P48 (at 136.4234 97.5614) (layer F.SilkS)
+    (effects (font (size 0.8 0.8) (thickness 0.15)))
+  )
+  (gr_text P49 (at 136.4234 95.0214) (layer F.SilkS)
+    (effects (font (size 0.8 0.8) (thickness 0.15)))
+  )
+  (gr_text P50 (at 136.4234 92.2274) (layer F.SilkS)
+    (effects (font (size 0.8 0.8) (thickness 0.15)))
+  )
+  (gr_text P51 (at 136.4234 89.6874) (layer F.SilkS)
+    (effects (font (size 0.8 0.8) (thickness 0.15)))
+  )
+  (gr_text P52 (at 136.4234 87.4014) (layer F.SilkS)
+    (effects (font (size 0.8 0.8) (thickness 0.15)))
+  )
+  (gr_text P53 (at 136.4234 84.6074) (layer F.SilkS)
+    (effects (font (size 0.8 0.8) (thickness 0.15)))
+  )
+  (gr_text P54 (at 136.4234 82.3214) (layer F.SilkS)
+    (effects (font (size 0.8 0.8) (thickness 0.15)))
+  )
+  (gr_text P55 (at 136.4234 79.7814) (layer F.SilkS)
+    (effects (font (size 0.8 0.8) (thickness 0.15)))
+  )
+  (gr_text P56 (at 136.6774 71.1454) (layer F.SilkS)
+    (effects (font (size 0.8 0.8) (thickness 0.15)))
+  )
+  (gr_text P57 (at 136.6774 68.6054) (layer F.SilkS)
+    (effects (font (size 0.8 0.8) (thickness 0.15)))
+  )
+  (gr_text P58 (at 136.6774 66.0654) (layer F.SilkS)
+    (effects (font (size 0.8 0.8) (thickness 0.15)))
+  )
+  (gr_text P59 (at 136.6774 63.5254) (layer F.SilkS)
+    (effects (font (size 0.8 0.8) (thickness 0.15)))
+  )
+  (gr_text P60 (at 136.6774 60.7314) (layer F.SilkS)
+    (effects (font (size 0.8 0.8) (thickness 0.15)))
+  )
+  (gr_text P61 (at 136.6774 58.1914) (layer F.SilkS)
+    (effects (font (size 0.8 0.8) (thickness 0.15)))
+  )
+  (gr_text P62 (at 136.6774 55.6514) (layer F.SilkS)
+    (effects (font (size 0.8 0.8) (thickness 0.15)))
+  )
+  (gr_text P63 (at 136.6774 53.1114) (layer F.SilkS)
+    (effects (font (size 0.8 0.8) (thickness 0.15)))
+  )
+  (gr_text 5V (at 156.4894 131.3434) (layer F.SilkS)
     (effects (font (size 1 1) (thickness 0.25)))
   )
-  (gr_text 3.3V (at 149.8854 77.4954) (layer F.Cu)
+  (gr_text 3.3V (at 150.1394 131.3434) (layer F.SilkS)
+    (effects (font (size 1 1) (thickness 0.25)))
+  )
+  (gr_text 3.3V (at 150.1394 103.9114) (layer F.SilkS)
+    (effects (font (size 1 1) (thickness 0.25)))
+  )
+  (gr_text 5V (at 156.4894 103.9114) (layer F.SilkS)
+    (effects (font (size 1 1) (thickness 0.25)))
+  )
+  (gr_text "S + -" (at 153.5504 126.5174) (layer F.SilkS)
+    (effects (font (size 1.25 1.25) (thickness 0.25)))
+  )
+  (gr_text "S + -" (at 153.5504 99.3394) (layer F.SilkS)
+    (effects (font (size 1.25 1.25) (thickness 0.25)))
+  )
+  (gr_text "S + -" (at 153.5504 73.1504) (layer F.SilkS)
+    (effects (font (size 1.25 1.25) (thickness 0.25)))
+  )
+  (gr_text 5V (at 156.2354 77.4954) (layer F.SilkS)
+    (effects (font (size 1 1) (thickness 0.25)))
+  )
+  (gr_text 3.3V (at 149.8854 77.4954) (layer F.SilkS)
     (effects (font (size 1 1) (thickness 0.25)))
   )
@@
     (effects (font (size 1 1) (thickness 0.15)))
   )
-  (gr_text "Propeller 2 Edge Breakout\nSonar Connect\nDPG 2025\nRev0" (at 94.7674 71.9074) (layer F.SilkS)
+  (gr_text "Propeller 2 Edge Breakout\nSonar Connect\nDPG 2025\nRev1" (at 94.7674 71.9074) (layer F.SilkS)
     (effects (font (size 1.5 1.5) (thickness 0.3)) (justify left))
   )
